Commit message: small changes

File: src/softleg_description/urdf/softlegisaac.urdf (robot description, URDF)
Before this commit: robot softlegisaac, 5 links, 4 joints
Links:
- removed link softleg_1_base_link
- removed link softleg_1_calf_link
- removed link softleg_1_cart_link
- removed link softleg_1_thigh_link
- added link base_link, mass 0.9724552; collision cylinder length=0.025 radius=0.035; visual mesh filename=package://softleg_description/meshes/base.stl scale=0.001 0.001 0.001
- added link calf_link, mass 0.0762175; collision sphere radius=0.015; visual mesh filename=package://softleg_description/meshes/calf.stl scale=0.001 0.001 0.001
- added link cart_link, mass 1e-4; visual mesh filename=package://softleg_description/meshes/cart.stl scale=0.001 0.001 0.001
- added link thigh_link, mass 0.435789; collision cylinder length=0.027 radius=0.03; visual mesh filename=package://softleg_description/meshes/thigh.stl scale=0.001 0.001 0.001
Joints:
- removed joint softleg_1_cart_joint
- removed joint softleg_1_hip_joint
- removed joint softleg_1_knee_joint
- added joint cart_joint: type prismatic, parent cart_link, child base_link, origin xyz=0. -0.005 0.0  rpy=3.1415927 -1.5707963 0. , axis 1 0 0, limit lower=0.0 upper=10.0 effort=500. velocity=1000.
- added joint hip_joint: type revolute, parent base_link, child thigh_link, origin xyz=0. -0.255 0.07  rpy=0. -1.5707963 0. , axis 1 0 0, limit lower=-3.1415927 upper=3.1415927 effort=100. velocity=57.6059555
- added joint knee_joint: type revolute, parent thigh_link, child calf_link, origin xyz=0.0275 -0.175 0.  rpy=1.5707964 0. 0. , axis 1 0 0, limit lower=-3.1415927 upper=3.1415927 effort=100. velocity=57.6059555
- joint fixed: child softleg_1_cart_link -> cart_link
